File: 6502_wozmon.kicad_pcb (KiCad board)
At the start: 2 copper layers, 186.8 x 132.7 mm, 38 parts, among them J1 Barrel_Jack_Switch_Pin3Ring, J2 DB9_Female, J3 "Switch", J4 Conn_01x08_Male, U1 7400, U2 W65C02, U3 28C256, U4 W65C51N, U5 62256, U6 MAX232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

Commit message: schematic updated to include debounced reset section; added barrel connector.
Parts:
- moved J1 59.2 mm to (33.3, 22.5), turned to -90 degrees
- moved J2 25.8 mm to (52.9, 21.2), turned to 180 degrees
Changed lines of the file:
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@@
     (fp_line (start -8.13 -2.64) (end -7.34 -2.64) (layer "F.SilkS") (width 0.12))
     (fp_arc (start 63.7 8) (mid 64.053553 8.146447) (end 64.2 8.5) (layer "F.SilkS") (width 0.12))
-    (fp_arc (start 64.20104 22.49932) (mid 64.054473 22.853115) (end 63.70066 22.9997) (layer "F.SilkS") (width 0.12))
+    (fp_arc (start 64.20104 22.49932) (mid 64.054479 22.85315) (end 63.70066 22.9997) (layer "F.SilkS") (width 0.12))
     (fp_arc (start 0.20066 22.9997) (mid -0.153162 22.853142) (end -0.29972 22.49932) (layer "F.SilkS") (width 0.12))
     (fp_arc (start -0.29972 8.49884) (mid -0.153162 8.145018) (end 0.20066 7.99846) (layer "F.SilkS") (width 0.12))
@@
   )
   (footprint "Connector_Dsub:DSUB-9_Female_Horizontal_P2.77x2.84mm_EdgePinOffset9.90mm_Housed_MountingHolesOffset11.32mm" (layer "F.Cu")
-    (at 39.010331 43.015 -90)
+    (at 52.87 21.230331 180)
     (descr "9-pin D-Sub connector, horizontal/angled (90 deg), THT-mount, female, pitch 2.77x2.84mm, pin-PCB-offset 9.9mm, distance of mounting holes 25mm, distance of mounting holes to PCB edge 11.32mm, see https://disti-assets.s3.amazonaws.com/tonar/files/datasheets/16730.pdf")
     (tags "9-pin D-Sub connector horizontal angled 90deg THT female pitch 2.77x2.84mm pin-PCB-offset 9.9mm mounting-holes-distance 25mm mounting-hole-offset 25mm")
@@
     (property "Sheetname" "")
     (attr through_hole)
-    (fp_text reference "J2" (at -5.54 -2.8 -90) (layer "F.SilkS")
-      (effects (font (size 1 1) (thickness 0.15)))
-    )
-    (fp_text value "DB9_Female" (at -5.54 20.81 -90) (layer "F.Fab")
-      (effects (font (size 1 1) (thickness 0.15)))
-    )
-    (fp_text user "${REFERENCE}" (at -5.54 16.225 -90) (layer "F.Fab")
+    (fp_text reference "J2" (at -5.54 -2.8) (layer "F.SilkS")
+      (effects (font (size 1 1) (thickness 0.15)))
+    )
+    (fp_text value "DB9_Female" (at -5.54 20.81) (layer "F.Fab")
+      (effects (font (size 1 1) (thickness 0.15)))
+    )
+    (fp_text user "${REFERENCE}" (at -5.54 16.225) (layer "F.Fab")
       (effects (font (size 1 1) (thickness 0.15)))
     )
@@
     (fp_arc (start 5.36 1.42) (mid 6.96 -0.18) (end 8.56 1.42) (layer "F.Fab") (width 0.1))
     (fp_arc (start -19.64 1.42) (mid -18.04 -0.18) (end -16.44 1.42) (layer "F.Fab") (width 0.1))
-    (pad "0" thru_hole circle (at -18.04 1.42 270) (size 4 4) (drill 3.2) (layers *.Cu *.Mask))
-    (pad "0" thru_hole circle (at 6.96 1.42 270) (size 4 4) (drill 3.2) (layers *.Cu *.Mask))
-    (pad "1" thru_hole rect (at 0 0 270) (size 1.6 1.6) (drill 1) (layers *.Cu *.Mask)
+    (pad "0" thru_hole circle (at -18.04 1.42 180) (size 4 4) (drill 3.2) (layers *.Cu *.Mask))
+    (pad "0" thru_hole circle (at 6.96 1.42 180) (size 4 4) (drill 3.2) (layers *.Cu *.Mask))
+    (pad "1" thru_hole rect (at 0 0 180) (size 1.6 1.6) (drill 1) (layers *.Cu *.Mask)
       (net 22 "unconnected-(J2-Pad1)") (pinfunction "1") (pintype "passive+no_connect"))
-    (pad "2" thru_hole circle (at -2.77 0 270) (size 1.6 1.6) (drill 1) (layers *.Cu *.Mask)
+    (pad "2" thru_hole circle (at -2.77 0 180) (size 1.6 1.6) (drill 1) (layers *.Cu *.Mask)
       (net 14 "RXD") (pinfunction "2") (pintype "passive"))
-    (pad "3" thru_hole circle (at -5.54 0 270) (size 1.6 1.6) (drill 1) (layers *.Cu *.Mask)
+    (pad "3" thru_hole circle (at -5.54 0 180) (size 1.6 1.6) (drill 1) (layers *.Cu *.Mask)
       (net 13 "TXD") (pinfunction "3") (pintype "passive"))
-    (pad "4" thru_hole circle (at -8.31 0 270) (size 1.6 1.6) (drill 1) (layers *.Cu *.Mask)
+    (pad "4" thru_hole circle (at -8.31 0 180) (size 1.6 1.6) (drill 1) (layers *.Cu *.Mask)
       (net 98 "unconnected-(J2-Pad4)") (pinfunction "4") (pintype "passive+no_connect"))
-    (pad "5" thru_hole circle (at -11.08 0 270) (size 1.6 1.6) (drill 1) (layers *.Cu *.Mask)
+    (pad "5" thru_hole circle (at -11.08 0 180) (size 1.6 1.6) (drill 1) (layers *.Cu *.Mask)
       (net 1 "GND") (pinfunction "5") (pintype "passive"))
-    (pad "6" thru_hole circle (at -1.385 2.84 270) (size 1.6 1.6) (drill 1) (layers *.Cu *.Mask)
+    (pad "6" thru_hole circle (at -1.385 2.84 180) (size 1.6 1.6) (drill 1) (layers *.Cu *.Mask)
       (net 99 "unconnected-(J2-Pad6)") (pinfunction "6") (pintype "passive+no_connect"))
-    (pad "7" thru_hole circle (at -4.155 2.84 270) (size 1.6 1.6) (drill 1) (layers *.Cu *.Mask)
+    (pad "7" thru_hole circle (at -4.155 2.84 180) (size 1.6 1.6) (drill 1) (layers *.Cu *.Mask)
       (net 100 "unconnected-(J2-Pad7)") (pinfunction "7") (pintype "passive+no_connect"))
-    (pad "8" thru_hole circle (at -6.925 2.84 270) (size 1.6 1.6) (drill 1) (layers *.Cu *.Mask)
+    (pad "8" thru_hole circle (at -6.925 2.84 180) (size 1.6 1.6) (drill 1) (layers *.Cu *.Mask)
       (net 101 "unconnected-(J2-Pad8)") (pinfunction "8") (pintype "passive+no_connect"))
-    (pad "9" thru_hole circle (at -9.695 2.84 270) (size 1.6 1.6) (drill 1) (layers *.Cu *.Mask)
+    (pad "9" thru_hole circle (at -9.695 2.84 180) (size 1.6 1.6) (drill 1) (layers *.Cu *.Mask)
       (net 102 "unconnected-(J2-Pad9)") (pinfunction "9") (pintype "passive+no_connect"))
     (model "${KICAD6_3DMODEL_DIR}/Connector_Dsub.3dshapes/DSUB-9_Female_Horizontal_P2.77x2.84mm_EdgePinOffset9.90mm_Housed_MountingHolesOffset11.32mm.wrl"
@@
   )
   (footprint "Connector_BarrelJack:BarrelJack_Horizontal" (layer "F.Cu")
-    (at 20.605 80.3225)
+    (at 33.3425 22.51 -90)
     (descr "DC Barrel Jack")
     (tags "Power Jack")
@@
     (property "Sheetname" "")
     (attr through_hole)
-    (fp_text reference "J1" (at -8.45 5.75) (layer "F.SilkS")
-      (effects (font (size 1 1) (thickness 0.15)))
-    )
-    (fp_text value "Barrel_Jack_Switch_Pin3Ring" (at -6.2 -5.5) (layer "F.Fab")
-      (effects (font (size 1 1) (thickness 0.15)))
-    )
-    (fp_text user "${REFERENCE}" (at -3 -2.95) (layer "F.Fab")
+    (fp_text reference "J1" (at -8.45 5.75 90) (layer "F.SilkS")
+      (effects (font (size 1 1) (thickness 0.15)))
+    )
+    (fp_text value "Barrel_Jack_Switch_Pin3Ring" (at -6.2 -5.5 90) (layer "F.Fab")
+      (effects (font (size 1 1) (thickness 0.15)))
+    )
+    (fp_text user "${REFERENCE}" (at -3 -2.95 90) (layer "F.Fab")
       (effects (font (size 1 1) (thickness 0.15)))
     )
@@
     (fp_line (start -13.7 -4.5) (end -13.7 4.5) (layer "F.Fab") (width 0.1))
     (fp_line (start -13.7 4.5) (end 0.8 4.5) (layer "F.Fab") (width 0.1))
-    (pad "1" thru_hole rect (at 0 0) (size 3.5 3.5) (drill oval 1 3) (layers *.Cu *.Mask)
+    (pad "1" thru_hole rect (at 0 0 270) (size 3.5 3.5) (drill oval 1 3) (layers *.Cu *.Mask)
       (net 3 "VCC") (pintype "passive"))
-    (pad "2" thru_hole roundrect (at -6 0) (size 3 3.5) (drill oval 1 3) (layers *.Cu *.Mask) (roundrect_rratio 0.25)
+    (pad "2" thru_hole roundrect (at -6 0 270) (size 3 3.5) (drill oval 1 3) (layers *.Cu *.Mask) (roundrect_rratio 0.25)
       (net 108 "unconnected-(J1-Pad2)") (pintype "passive+no_connect"))
-    (pad "3" thru_hole roundrect (at -3 4.7) (size 3.5 3.5) (drill oval 3 1) (layers *.Cu *.Mask) (roundrect_rratio 0.25)
+    (pad "3" thru_hole roundrect (at -3 4.7 270) (size 3.5 3.5) (drill oval 3 1) (layers *.Cu *.Mask) (roundrect_rratio 0.25)
       (net 1 "GND") (pintype "passive"))
     (model "${KICAD6_3DMODEL_DIR}/Connector_BarrelJack.3dshapes/BarrelJack_Horizontal.wrl"

Commit message: increment
Parts:
- removed LED_3, LED_4: LED, LED_THT:LED_D5.0mm
- removed R8: 220, Resistor_THT:R_Axial_DIN0207_L6.3mm_D2.5mm_P10.16mm_Horizontal
- added C10: C, Capacitor_THT:C_Disc_D5.0mm_W2.5mm_P5.00mm, F.Cu at (56.5, 59.1)
- added C11: 10u, Capacitor_THT:C_Disc_D5.0mm_W2.5mm_P5.00mm, F.Cu at (60.3, 59.1)
- added D3: LED, LED_THT:LED_D5.0mm, F.Cu at (57.3, 33.0)
- added J5: Conn_01x03_Male, Connector_PinHeader_2.54mm:PinHeader_1x03_P2.54mm_Vertical, F.Cu at (45.1, 30.5)
- added R6: 1K, Resistor_THT:R_Axial_DIN0207_L6.3mm_D2.5mm_P10.16mm_Horizontal, F.Cu at (56.5, 55.9)
- added U9: 74HC14, Package_DIP:DIP-14_W7.62mm_Socket, F.Cu at (41.4, 46.4)
- C1: value 0.1u -> C
- J3: value "Switch" -> Conn_01x03_Male
- R1: value 1K -> 10K
- R7: value 220 -> 330
- moved G*** 60.7 mm to (160.7, 90.8)
- moved C1 57.3 mm to (52.7, 59.1), turned to -90 degrees
- moved R7 28.7 mm to (60.3, 45.7)
- moved LED_1 27.9 mm to (33.0, 32.4)
- moved LED_2 27.8 mm to (33.0, 40.6)
- moved R1 26.1 mm to (52.7, 55.9)
- moved J3 25.2 mm to (45.1, 38.1), turned to 90 degrees
- moved J1 2.25 mm to (33.3, 24.8)
Connections:
- C1 pad 1: GND -> VCC
- C1 pad 2: Net-(C1-Pad2) -> GND
- J3 pad 2: RESET* -> unconnected-(J3-Pad2)
- J3 pad 3: Net-(C1-Pad2) -> unconnected-(J3-Pad3)
- J4 pad 1: GND -> CLK
- J4 pad 2: GND -> RESET*
- J4 pad 3: GND -> MAX232_12
- J4 pad 4: GND -> TXD
- J4 pad 5: CLK -> GND
- J4 pad 6: XTAL -> GND
- J4 pad 7: unconnected-(J4-Pad7) -> GND
- J4 pad 8: unconnected-(J4-Pad8) -> GND
- R1 pad 1: VCC -> Net-(J5-Pad1)
- R1 pad 2: Net-(J3-Pad1) -> VCC
- U4 pad 12: Net-(R7-Pad1) -> MAX232_12
- U6 pad 12: Net-(R7-Pad1) -> MAX232_12
Routing:
- net TXD: track 50.2 -> 168.5 mm, vias 0 -> 1
- net MAX232_12: track 0.00 -> 86.4 mm, vias 0 -> 1
- net RESET*: track 156.2 -> 221.1 mm, vias 3 -> 5
- net VCC: track 450.3 -> 511.9 mm, vias 7 -> 9
- net Net-(C1-Pad2): track 57.5 -> 0.00 mm, vias 1 -> 0
- net Net-(R7-Pad1): track 82.9 -> 26.0 mm, vias 2 -> 0
- net Net-(U4-Pad10): track 82.9 -> 48.3 mm, vias 3 -> 1
- net Net-(C11-Pad1): track 0.00 -> 33.6 mm
- net RXD: track 42.8 -> 76.3 mm, vias 0 -> 1
- net Net-(LED_4-Pad2): track 32.8 -> 0.00 mm, vias 1 -> 0
- net Net-(J5-Pad1): track 0.00 -> 31.2 mm, vias 0 -> 1
- net XTAL: track 46.5 -> 31.7 mm
- net Net-(LED_2-Pad2): track 49.4 -> 39.9 mm, vias 1 -> 0
- net Net-(J3-Pad1): track 18.7 -> 26.8 mm
- net GND: track 557.1 -> 563.9 mm, vias 11 -> 9
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Other:
- board size 186.8 x 132.7 mm -> 186.3 x 130.3 mm
- board text added: "0000 A9 01 0002 18 0003 69 01 0005 85 08 0007 4C 00 FF"
- board text added: "0x0000 - 0x00FF ZP 0x0100 - 0x01FF STACK 0x0200 - 0x3FFF USER 0x4000 - 0x4FFF UNUSED 0x5000 - 0x5003 ACIA 0x6000 - 0x600F VIA 0x7000 - 0x7FFF UNUSED 0x8000 - 0xFFFF ROM WOZMON: FF00"
- board text added: "28C256 ROM"
- board text added: "62256 RAM"
- board text added: "6502"
- board text added: "65c02"
- board text added: "; ASM DIRECTIVES ... ; MAIN .org $8000 reset: ... nmi: RTI ; RESET/IRQ VECTORS .org $FFFA .word nmi .word reset .word $0000"
- board text added: "= $6000 = $6001 = $6002 = $6003"
- board text added: "BASED ON THE ORIGINAL"
- board text added: "BAUD RATE: 19200 8N1 RAM: 0x0000 - 0x7FFF ROM: 0x8000 - 0xFFFF"
- board text added: "LDA #$01 CLC ADC #$01 STA $0008 JMP $FF00"
- board text added: "MAX232_12"
- board text added: "N V B D I Z C"
- board text added: "PATH/vasm6502_oldstyle -c02 -Fbin -dotdir -o f.bin -L f.lst f.s PATH/minipro -p AT28C256 -w f.bin"
- board text added: "PCB: TIM SANDERS"
- board text added: "PORTB PORTA DDRB DDRB"
- board text added: "PROCESSOR: 65C02 CLOCK: 1MHZ HORZ: 200NSEC"
- board text added: "RESET*"
- board text added: "REV: JUL 2024 SCHEMATIC: 6502_WOZMON.KICAD_SCH SPECIAL THANKS TO BEN EATER"
- board text added: "TXD"
- board text added: "| NEGATIVE | OVERFLOW | BRK INSTR | DECIMAL MODE | IRQ DISABLE | ZERO | CARRY"
- board text removed: "+5"
- board text removed: "28C256 RAM"
- board text removed: "62256 ROM"
- board text removed: "65C02"
- board text removed: "65C02 1 MHZ 8 BITS 16 BITS"
- board text removed: "F=1MHZ, HORZ=200NSEC"
- board text removed: "NC"
- board text removed: "OUTPUT"
- board text removed: "PCB: TIM SANDERS, FEB 2024 SPECIAL THANKS TO BEN EATER"
- board text removed: "PROCESSOR: CLOCK SPEED: DATA BUS: ADDRESS BUS:"
- board text removed: "RxD"
- board text removed: "TxD"
- board text removed: "XTL"

Commit message: 1.  Updated Files     A.  The pin headers being used as a switch were replaced with a proper button switch and footprint.         a.  The following were updated:             1.  6502_wozmon.kicad_pcb 	        2.  6502_wozmon.kicad_prl 2.  Notes     A.  The silkscreen for the RAM and ROM chips is reversed.         a.  This is becuase the footprints are reversed in the schematic editor.             1.  I switched the footprints, but this caused *37& clearance violations in the PCB editor.             2.  Fixing this would have required *substantial* re-routing.             3.  I decided for forego fixing this; I will accept this minor issue on the silkscreen.
Parts:
- removed J3, J5: Conn_01x03_Male, Connector_PinHeader_2.54mm:PinHeader_1x03_P2.54mm_Vertical
- added SW2: SW_Push_Dual, Button_Switch_THT:SW_Tactile_Straight_KSA0Axx1LFTR, F.Cu at (50.3, 30.5)
Routing:
- net Net-(R1-Pad1): track 31.2 -> 22.6 mm
- net Net-(R6-Pad1): track 26.8 -> 32.1 mm
- net GND: track 563.9 -> 563.2 mm, vias 9 -> 11
Other:
- board text added: "REV: 21 JUL 2024 SCHEMATIC: 6502_WOZMON.KICAD_SCH BRANCH: 20240720 SPECIAL THANKS TO BEN EATER"
- board text removed: "REV: JUL 2024 SCHEMATIC: 6502_WOZMON.KICAD_SCH SPECIAL THANKS TO BEN EATER"

Commit message: Added gerber files.
Other:
- board size 186.3 x 130.3 mm -> 183.7 x 131.3 mm
- board text added: "0x0000-0x00FF ZERO 0x0100-0x01FF STACK 0x0200-0x3FFF USER 0x4000-0x4FFF UNUSED 0x5000-0x5003 ACIA 0x6000-0x600F VIA 0x7000-0x7FFF UNUSED 0x8000-0xFFFF ROM 0x6000 | IRB / ORB 0x6001 | IRA / ORA 0x6002 | DDRB 0x6003 | DDRA WOZMON \ FF00 R ; MAIN .org $8000 RESET: ... ; SUBROUTINES ... NMI: RTI ; RESET/IRQ VECTORS .org $FFFA .word NMI .word RESET .word $0000"
- board text added: "65C51 ACIA / UART"
- board text added: "7414"
- board text added: "8-BIT 65c02 COMPUTER"
- board text added: "CS0"
- board text added: "CS1B"
- board text added: "CTSB"
- board text added: "DCDB"
- board text added: "DSRB"
- board text added: "DTRB"
- board text added: "IRQB"
- board text added: "OUTPUT"
- board text added: "PCB DESIGNED BY TIM SANDERS https://github.com/tsanders30004"
- board text added: "RTSB"
- board text added: "RW*"
- board text added: "RxC"
- board text added: "RxD"
- board text added: "SCHEMATIC: 6502_WOZMON.KICAD_SCH BRANCH: 20240720 PROCESSOR: 65C02 CLOCK: 1MHZ HORZ: 200NSEC"
- board text added: "SPECIAL THANKS TO BEN EATER https://eater.net"
- board text added: "TxD"
- board text added: "XLTO"
- board text added: "XTLI"
- board text removed: "0000 A9 01 0002 18 0003 69 01 0005 85 08 0007 4C 00 FF"
- board text removed: "0x0000 - 0x00FF ZP 0x0100 - 0x01FF STACK 0x0200 - 0x3FFF USER 0x4000 - 0x4FFF UNUSED 0x5000 - 0x5003 ACIA 0x6000 - 0x600F VIA 0x7000 - 0x7FFF UNUSED 0x8000 - 0xFFFF ROM WOZMON: FF00"
- board text removed: "65C51 UART"
- board text removed: "65c02"
- board text removed: "; ASM DIRECTIVES ... ; MAIN .org $8000 reset: ... nmi: RTI ; RESET/IRQ VECTORS .org $FFFA .word nmi .word reset .word $0000"
- board text removed: "= $6000 = $6001 = $6002 = $6003"
- board text removed: "LDA #$01 CLC ADC #$01 STA $0008 JMP $FF00"
- board text removed: "N V B D I Z C"
- board text removed: "PATH/vasm6502_oldstyle -c02 -Fbin -dotdir -o f.bin -L f.lst f.s PATH/minipro -p AT28C256 -w f.bin"
- board text removed: "PCB: TIM SANDERS"
- board text removed: "PORTB PORTA DDRB DDRB"
- board text removed: "PROCESSOR: 65C02 CLOCK: 1MHZ HORZ: 200NSEC"
- board text removed: "REV: 21 JUL 2024 SCHEMATIC: 6502_WOZMON.KICAD_SCH BRANCH: 20240720 SPECIAL THANKS TO BEN EATER"
- board text removed: "| NEGATIVE | OVERFLOW | BRK INSTR | DECIMAL MODE | IRQ DISABLE | ZERO | CARRY"

Commit message: Added README.md, photos, and sotware files.
Connections:
- J1 pad 2: unconnected-(J1-Pad2) -> GND
- SW2 pad 2: GND -> Net-(R6-Pad1)
- SW2 pad 3: Net-(R6-Pad1) -> GND
Routing:
- net GND: track 563.2 -> 559.2 mm, vias 11 -> 10
- net Net-(R6-Pad1): track 32.1 -> 35.9 mm
Other:
- board text added: "0x0000-0x00FF ZERO 0x0100-0x01FF STACK 0x0200-0x3FFF USER 0x4000-0x4FFF UNUSED 0x5000-0x5003 ACIA 0x6000-0x600F VIA 0x7000-0x7FFF UNUSED 0x8000-0xFFFF ROM"
- board text added: "0x6000 | IRB/ORB 0x6001 | IRA/ORA 0x6002 | DDRB 0x6003 | DDRA WOZMON \ FF00 R ; MAIN .org $8000 RESET: ... ; SUBROUTINES ... NMI: RTI ; RESET/IRQ VEC .org $FFFA .word NMI .word RESET .word $0000"
- board text added: "28C256 RAM"
- board text added: "65c02"
- board text added: "ADDRESS DECODING"
- board text added: "INVERTER FOR RESET DEBOUNCE"
- board text added: "RAM"
- board text added: "ROM"
- board text added: "SCHEMATIC: 6502_WOZMON.KICAD_SCH BRANCH: 20240818 PROCESSOR: 65C02 CLOCK: 1MHZ HORZ: 200NSEC"
- board text removed: "0x0000-0x00FF ZERO 0x0100-0x01FF STACK 0x0200-0x3FFF USER 0x4000-0x4FFF UNUSED 0x5000-0x5003 ACIA 0x6000-0x600F VIA 0x7000-0x7FFF UNUSED 0x8000-0xFFFF ROM 0x6000 | IRB / ORB 0x6001 | IRA / ORA 0x6002 | DDRB 0x6003 | DDRA WOZMON \ FF00 R ; MAIN .org $8000 RESET: ... ; SUBROUTINES ... NMI: RTI ; RESET/IRQ VECTORS .org $FFFA .word NMI .word RESET .word $0000"
- board text removed: "28C256 ROM"
- board text removed: "SCHEMATIC: 6502_WOZMON.KICAD_SCH BRANCH: 20240720 PROCESSOR: 65C02 CLOCK: 1MHZ HORZ: 200NSEC"

Commit message: Add files via upload
Other:
- board text added: "SCHEMATIC: 6502_WOZMON.KICAD_SCH BRANCH: 20250121 PROCESSOR: 65C02 CLOCK: 1MHZ HORZ: 200NSEC"
- board text removed: "PCB DESIGNED BY TIM SANDERS https://github.com/tsanders30004"
- board text removed: "SCHEMATIC: 6502_WOZMON.KICAD_SCH BRANCH: 20240818 PROCESSOR: 65C02 CLOCK: 1MHZ HORZ: 200NSEC"
Changed lines of the file:
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@@
     (effects (font (size 1 1) (thickness 0.15)) (justify left))
-  )
-  (gr_text "PCB DESIGNED BY TIM SANDERS\nhttps://github.com/tsanders30004" (at 113.792 136.652) (layer "F.SilkS")
-    (effects (font (size 1.524 1.524) (thickness 0.2794)) (justify left))
   )
   (gr_text "A12" (at 135.89 44.459769) (layer "F.SilkS")
@@
     (effects (font (size 1 1) (thickness 0.15)) (justify left))
   )
-  (gr_text "SCHEMATIC: 6502_WOZMON.KICAD_SCH\nBRANCH:  20240818\n\nPROCESSOR: 65C02\nCLOCK:  1MHZ\nHORZ:   200NSEC\n" (at 77.724 19.37258) (layer "F.SilkS")
+  (gr_text "SCHEMATIC: 6502_WOZMON.KICAD_SCH\nBRANCH:    20250121\n\nPROCESSOR: 65C02\nCLOCK:  1MHZ\nHORZ:   200NSEC\n" (at 77.724 19.37258) (layer "F.SilkS")
     (effects (font (size 1.524 1.524) (thickness 0.2794)) (justify left))
   )
